File: palscope.kicad_sch (KiCad schematic)
At the start: 39 parts, among them J1 Conn_Coaxial, J2 Y, J3 Z, J4 X, J5 CVcc, J6 CGND, Q1 2N3906, Q2 2N3904, Q3 2N3906, Q4 2N3904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

Commit message: reworked PCB, removed useless connections, fixed bad C6 capacity
Parts:
- C6: value 0.01n -> 0.01u
- J1: footprint Connector_Coaxial:MMCX_Molex_73415-0961_Horizontal_0.8mm-PCB -> Connector:CUI_RCJ-013
Connections:
- net GND: no longer U1.5 (BURST), U1.7 (O/E)
Other:
- company: (none) -> Thomas Lecomte - thomas@netnix.in
- title: (none) -> PAL to X-Y-Z Raster
- moved on the sheet: D1, D2, J4, Q6, R10, R11, R12, R4, R9
